File: mu-kb.kicad_pcb (KiCad board)
At the start: 2 copper layers, 239.5 x 92.5 mm, 80 parts, among them SW1 SW_Push_45deg, SW10 SW_Push_45deg, SW11 SW_Push_45deg, SW12 SW_Push_45deg, SW13 SW_Push_45deg, SW14 SW_Push_45deg, SW15 SW_Push_45deg, SW16 SW_Push_45deg, SW17 SW_Push_45deg, SW18 SW_Push_45deg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

Commit message: completed v2
Parts:
- moved R_U1 1.00 mm to (159.5, 79.0), turned to 0 degrees
- moved U1 1.00 mm to (137.5, 79.0), turned to 0 degrees
Routing:
- net Col0: track 0.00 -> 161.5 mm, vias 0 -> 15
- net Col2: track 0.00 -> 153.5 mm, vias 0 -> 18
- net R_Col4: track 0.00 -> 148.3 mm, vias 0 -> 12
- net Row0: track 0.00 -> 147.7 mm, vias 0 -> 19
- net Row1: track 0.00 -> 141.2 mm, vias 0 -> 11
- net R_Row0: track 0.00 -> 136.8 mm, vias 0 -> 6
- net Col1: track 0.00 -> 135.0 mm, vias 0 -> 13
- net R_Col2: track 0.00 -> 132.9 mm, vias 0 -> 10
- net Col3: track 0.00 -> 131.9 mm, vias 0 -> 12
- net R_Col3: track 0.00 -> 122.0 mm, vias 0 -> 10
- net Row2: track 0.00 -> 119.5 mm, vias 0 -> 12
- net Col4: track 0.00 -> 116.3 mm, vias 0 -> 12
- net R_Row2: track 0.00 -> 113.9 mm, vias 0 -> 8
- net R_Row3: track 0.00 -> 110.8 mm, vias 0 -> 10
- net R_Col1: track 0.00 -> 109.1 mm, vias 0 -> 10
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- added copper zone on B.Cu, net GND
- added copper zone on F.Cu, net GND
